File: pcbV4.kicad_pcb (KiCad board)
At the start: 4 copper layers, 59.4 x 30 mm, 68 parts, among them J3 NRESET, Q1 DMC2400UV-7, U1 LSM6DSOXTR, U2 MAX30001CWV+T, U4 NPM1100-QDAA-R, U6 TLV70018DCKR, U9 W25Q256JVEIQTR

Commit message: Update PCB design
Parts:
- renumbered GND to J4, VDD to J5, SCLK to J6, SWDIO to J7, BTN to SW1, SHPACT to TP1, FCLK to TP2, MISO to TP3, MOSI to TP4
Connections:
- LED1 pad 2: Net-(LED1-G-) -> VDD
- LED1 pad 4: VDD -> Net-(LED1-+)
- R18 pad 1: Net-(LED1-G-) -> Net-(LED1-+)
- USB2 pad A9: unconnected-(USB2-VBUS-PadA9) -> VBUS
Routing:
- net GND: track 104.0 -> 112.1 mm, vias 26 -> 28
- net Net-(LED1-+): track 0.00 -> 1.51 mm
- net MOSI: track 42.7 -> 44.1 mm
- net Net-(LED1-G-): track 1.14 -> 0.00 mm
- net MISO: track 50.5 -> 51.2 mm
- net VDD: track 114.6 -> 113.9 mm
- net FCLK: vias 5 -> 4
