File: pcbV4.kicad_sch (KiCad schematic)
At the start: 54 parts, among them J3 GND, J4 GND, J5 VDD, J6 SWDCLK, J7 SWDIO, SW1 XDMK-12C01-25, U1 LSM6DSOXTR, U2 MAX30001CWV+T, U4 NPM1100-QDAA-R, U5 BS-08-B2AA020-R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

Commit message: Update pcbV4 schematic
Parts:
- removed LED1, LED2: Blue light 0603, easyeda2kicad:LED0603-RD, symbol easyeda2kicad:Bluelight0603
- removed SW1: XDMK-12C01-25, easyeda2kicad:SW-SMD_XDMK-12C01-25, symbol easyeda2kicad:XDMK-12C01-25
- added C27: 100nF, symbol Device:C
- added Q1: DMC2400UV-7, easyeda2kicad:SOT-563_L1.6-W1.2-P0.50-LS1.6-BL, symbol battery:DMC2400UV-7
- added R12: 1M5, symbol Device:R
- added R13: 220k, symbol Device:R
- added R14: 1M, symbol Device:R
- added TP1: TestPoint, symbol Connector:TestPoint
- added U7: W25Q256JVFIQT, easyeda2kicad:SOIC-16_L10.3-W7.5-P1.27-LS10.3-BL, symbol battery:W25Q256JVFIQT
- R11: value 4k7 -> 1M; footprint Resistor_SMD:R_0402_1005Metric -> (none)
- R3, R4: value 200k -> 200
- R9: value 1k5 -> 14k
Connections:
- net VOUT is gone; now on net VDD: C21.1, L1.1, U4.1 (VOUTB)
- net GND: now also C27.2, Q1.1 (S1), R13.2, U7.10 (GND); no longer U4.6 (SHPACT)
- net MISO: now also U7.8 (DO(IO1))
- net MOSI: now also U7.15 (DI(IO0))
- net SCLK: now also U7.16 (CLK)
- net VDD: now also C27.1, U7.1 (RESET#(IO3)), U7.2 (VCC), U7.3 (~{RESET}), U7.9 (WP#(IO2))
- net bat+: now also Q1.4 (S2), R14.2
- net BAT_MON_EN: now reaches R11.1
- net BAT_MON_EN: now also Q1.2 (G1)
- new net: Q1.5 (G2), Q1.6 (D1), R14.1
- new net: Q1.3 (D2), R12.1
- new net BAT_MON: R12.2, R13.1
- new net SHPACT: TP1.1, U4.6 (SHPACT)
- new net W25_CS: U7.7 (~{CS})
- no-connect marks 18 -> 22
Other:
- note added: "Bat voltage = BAT_MON / 0.1279"
- note added: "Battery monitoring circuit"
- note added: "NOR Flash"
- moved on the sheet: BB1, C10, C11, C12, C13, C14, C15, C16, C18, C19, C2, C20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

Commit message: Update pcbV4 schematic
Parts:
- added C28: 0.01uF, symbol Device:C
- added OSC1: SX2M32.768KM20F30TNN, easyeda2kicad:OSC-SMD_4P-L2.5-W2.0-BL, symbol battery:SX2M32.768KM20F30TNN
- added TP2: TestPoint, symbol Connector:TestPoint
Connections:
- net FCLK: now also OSC1.3 (OUTPUT), TP2.1; no longer U3.16 (P1.08)
- net GND: now also C28.1, OSC1.2 (GND)
- net VDD: now also C28.2, OSC1.4 (VDD)
- no-connect marks 22 -> 23
Other:
- note added: "Crystal Oscillator 32.668KHz"
Changed lines of the file:
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@@
   (junction (at 108.585 41.91) (diameter 0) (color 0 0 0 0)
   )
+  (junction (at 126.365 149.86) (diameter 0) (color 0 0 0 0)
+  )
+  (junction (at 120.65 147.32) (diameter 0) (color 0 0 0 0)
+  )
   (junction (at 54.61 223.52) (diameter 0) (color 0 0 0 0)
   )
@@
   (no_connect (at 307.34 49.53))
   (no_connect (at 375.92 121.92))
+  (no_connect (at 80.01 147.32))
   (no_connect (at 266.7 44.45))
   (no_connect (at 93.98 36.83))
@@
     (stroke (width 0) (type default))
   )
+  (wire (pts (xy 76.835 149.86) (xy 80.01 149.86))
+    (stroke (width 0) (type default))
+  )
   (wire (pts (xy 179.07 46.99) (xy 184.15 46.99))
     (stroke (width 0) (type default))
@@
     (stroke (width 0) (type default))
   )
+  (wire (pts (xy 120.65 149.86) (xy 126.365 149.86))
+    (stroke (width 0) (type default))
+  )
   (wire (pts (xy 73.66 261.62) (xy 73.66 262.89))
     (stroke (width 0) (type default))
@@
     (stroke (width 0) (type default))
   )
+  (wire (pts (xy 120.65 144.78) (xy 120.65 147.32))
+    (stroke (width 0) (type default))
+  )
   (wire (pts (xy 46.99 240.03) (xy 54.61 240.03))
     (stroke (width 0) (type default))
@@
     (stroke (width 0) (type default))
   )
+  (wire (pts (xy 120.65 147.32) (xy 123.19 147.32))
+    (stroke (width 0) (type default))
+  )
   (wire (pts (xy 163.83 16.51) (xy 167.64 16.51))
     (stroke (width 0) (type default))
@@
     (stroke (width 0) (type default))
   )
-  (wire (pts (xy 179.07 57.15) (xy 183.515 57.15))
-    (stroke (width 0) (type default))
-  )
   (wire (pts (xy 179.07 41.91) (xy 184.15 41.91))
     (stroke (width 0) (type default))
@@
     (stroke (width 0) (type default))
   )
+  (wire (pts (xy 126.365 149.86) (xy 133.35 149.86))
+    (stroke (width 0) (type default))
+  )
   (wire (pts (xy 77.47 177.8) (xy 83.185 177.8))
     (stroke (width 0) (type default))
@@
     (fill (type none))
   )
+  (rectangle (start 69.85 133.985) (end 143.51 158.115)
+    (stroke (width 0) (type default))
+    (fill (type none))
+  )
   (rectangle (start 309.245 196.215) (end 395.605 245.11)
     (stroke (width 0) (type default))
@@
     (effects (font (size 1.27 1.27)) (justify left bottom))
   )
+  (text "Crystal Oscillator 32.668KHz" (at 72.39 137.16 0)
+    (effects (font (size 1.27 1.27)) (justify left bottom))
+  )
   (text "32.768kHz" (at 123.825 227.33 0)
     (effects (font (size 1.27 1.27)) (justify left bottom))
@@
     (effects (font (size 1.27 1.27)) (justify left bottom))
   )
-  (text "32.768kHz" (at 191.77 57.785 0)
-    (effects (font (size 1.27 1.27)) (justify left bottom))
-  )
   (text "NPM1100" (at 205.105 198.755 0)
     (effects (font (size 1.27 1.27)) (justify left bottom))
@@
     (effects (font (size 1.27 1.27)) (justify left bottom))
   )
+  (text "32.768kHz" (at 125.73 153.035 0)
+    (effects (font (size 1.27 1.27)) (justify left bottom))
+  )
   (text "Battery" (at 346.075 25.4 0)
     (effects (font (size 1.27 1.27)) (justify left bottom))
@@
     )
   )
+  (global_label "FCLK" (shape input) (at 133.35 149.86 0) (fields_autoplaced)
+    (effects (font (size 1.27 1.27)) (justify left))
+    (property "Intersheetrefs" "${INTERSHEET_REFS}" (at 140.6254 149.86 0)
+      (effects (font (size 1.27 1.27)) (justify left) hide)
+    )
+  )
   (global_label "MISO" (shape input) (at 183.515 39.37 0) (fields_autoplaced)
     (effects (font (size 1.27 1.27)) (justify left))
@@
     )
   )
-  (global_label "FCLK" (shape input) (at 183.515 57.15 0) (fields_autoplaced)
-    (effects (font (size 1.27 1.27)) (justify left))
-    (property "Intersheetrefs" "${INTERSHEET_REFS}" (at 190.7904 57.15 0)
-      (effects (font (size 1.27 1.27)) (justify left) hide)
-    )
-  )
   (global_label "VSYS" (shape input) (at 228.6 222.885 180) (fields_autoplaced)
     (effects (font (size 1.27 1.27)) (justify right))
@@
     )
   )
+  (symbol (lib_id "battery:SX2M32.768KM20F30TNN") (at 100.33 148.59 0) (unit 1)
+    (in_bom yes) (on_board yes) (dnp no) (fields_autoplaced)
+    (property "Reference" "OSC1" (at 100.33 140.335 0)
+      (effects (font (size 1.27 1.27)))
+    )
+    (property "Value" "SX2M32.768KM20F30TNN" (at 100.33 142.875 0)
+      (effects (font (size 1.27 1.27)))
+    )
+    (property "Footprint" "easyeda2kicad:OSC-SMD_4P-L2.5-W2.0-BL" (at 100.33 157.48 0)
+      (effects (font (size 1.27 1.27)) hide)
+    )
+    (property "Datasheet" "https://www.lcsc.com/datasheet/C2901603.pdf" (at 100.33 160.02 0)
+      (effects (font (size 1.27 1.27)) hide)
+    )
+    (property "Manufacturer" "SCTF(星通时频)" (at 100.33 162.56 0)
+      (effects (font (size 1.27 1.27)) hide)
+    )
+    (property "MPN" "SX2M32.768KM20F30TNN" (at 100.33 165.1 0)
+      (effects (font (size 1.27 1.27)) hide)
+    )
+    (property "LCSC Part" "C2901603" (at 100.33 167.64 0)
+      (effects (font (size 1.27 1.27)) hide)
+    )
+    (pin "1")
+    (pin "2")
+    (pin "3")
+    (pin "4")
+    (instances
+      (project "pcbV4"
+        (path "/499be7d4-fba5-4711-ae03-4b2682fa02d7"
+          (reference "OSC1") (unit 1)
+        )
+      )
+    )
+  )
   (symbol (lib_id "Device:R") (at 62.865 262.89 90) (unit 1)
     (in_bom yes) (on_board yes) (dnp no) (fields_autoplaced)
@@
     )
   )
+  (symbol (lib_id "Connector:TestPoint") (at 126.365 149.86 0) (unit 1)
+    (in_bom yes) (on_board yes) (dnp no) (fields_autoplaced)
+    (property "Reference" "TP2" (at 128.905 145.2879 0)
+      (effects (font (size 1.27 1.27)) (justify left))
+    )
+    (property "Value" "TestPoint" (at 128.905 147.8279 0)
+      (effects (font (size 1.27 1.27)) (justify left))
+    )
+    (property "Footprint" "" (at 131.445 149.86 0)
+      (effects (font (size 1.27 1.27)) hide)
+    )
+    (property "Datasheet" "~" (at 131.445 149.86 0)
+      (effects (font (size 1.27 1.27)) hide)
+    )
+    (pin "1")
+    (instances
+      (project "pcbV4"
+        (path "/499be7d4-fba5-4711-ae03-4b2682fa02d7"
+          (reference "TP2") (unit 1)
+        )
+      )
+    )
+  )
   (symbol (lib_id "Device:C") (at 113.665 237.49 0) (unit 1)
     (in_bom yes) (on_board yes) (dnp no) (fields_autoplaced)
@@
     )
   )
+  (symbol (lib_id "power:GND") (at 120.65 137.16 180) (unit 1)
+    (in_bom yes) (on_board yes) (dnp no) (fields_autoplaced)
+    (property "Reference" "#PWR058" (at 120.65 130.81 0)
+      (effects (font (size 1.27 1.27)) hide)
+    )
+    (property "Value" "GND" (at 120.65 132.08 0)
+      (effects (font (size 1.27 1.27)))
+    )
+    (property "Footprint" "" (at 120.65 137.16 0)
+      (effects (font (size 1.27 1.27)) hide)
+    )
+    (property "Datasheet" "" (at 120.65 137.16 0)
+      (effects (font (size 1.27 1.27)) hide)
+    )
+    (pin "1")
+    (instances
+      (project "pcbV4"
+        (path "/499be7d4-fba5-4711-ae03-4b2682fa02d7"
+          (reference "#PWR058") (unit 1)
+        )
+      )
+    )
+  )
   (symbol (lib_id "Connector:Conn_01x01_Pin") (at 372.11 80.645 180) (unit 1)
     (in_bom yes) (on_board yes) (dnp no)
@@
     )
   )
+  (symbol (lib_id "power:VDD") (at 123.19 147.32 0) (unit 1)
+    (in_bom yes) (on_board yes) (dnp no)
+    (property "Reference" "#PWR057" (at 123.19 151.13 0)
+      (effects (font (size 1.27 1.27)) hide)
+    )
+    (property "Value" "VDD" (at 125.095 144.78 0)
+      (effects (font (size 1.27 1.27)))
+    )
+    (property "Footprint" "" (at 123.19 147.32 0)
+      (effects (font (size 1.27 1.27)) hide)
+    )
+    (property "Datasheet" "" (at 123.19 147.32 0)
+      (effects (font (size 1.27 1.27)) hide)
+    )
+    (pin "1")
+    (instances
+      (project "pcbV4"
+        (path "/499be7d4-fba5-4711-ae03-4b2682fa02d7"
+          (reference "#PWR057") (unit 1)
+        )
+      )
+    )
+  )
   (symbol (lib_id "power:GND") (at 277.495 235.585 0) (unit 1)
     (in_bom yes) (on_board yes) (dnp no) (fields_autoplaced)
@@
     )
   )
+  (symbol (lib_id "power:GND") (at 76.835 149.86 0) (unit 1)
+    (in_bom yes) (on_board yes) (dnp no) (fields_autoplaced)
+    (property "Reference" "#PWR056" (at 76.835 156.21 0)
+      (effects (font (size 1.27 1.27)) hide)
+    )
+    (property "Value" "GND" (at 76.835 154.305 0)
+      (effects (font (size 1.27 1.27)))
+    )
+    (property "Footprint" "" (at 76.835 149.86 0)
+      (effects (font (size 1.27 1.27)) hide)
+    )
+    (property "Datasheet" "" (at 76.835 149.86 0)
+      (effects (font (size 1.27 1.27)) hide)
+    )
+    (pin "1")
+    (instances
+      (project "pcbV4"
+        (path "/499be7d4-fba5-4711-ae03-4b2682fa02d7"
+          (reference "#PWR056") (unit 1)
+        )
+      )
+    )
+  )
   (symbol (lib_id "power:VDD") (at 311.15 54.61 180) (unit 1)
     (in_bom yes) (on_board yes) (dnp no)
@@
         )
       )
+    )
+  )
+  (symbol (lib_id "Device:C") (at 120.65 140.97 0) (unit 1)
+    (in_bom yes) (on_board yes) (dnp no) (fields_autoplaced)
+    (property "Reference" "C28" (at 124.46 139.6999 0)
+      (effects (font (size 1.27 1.27)) (justify left))
+    )
+    (property "Value" "0.01uF" (at 124.46 142.2399 0)
+      (effects (font (size 1.27 1.27)) (justify left))
+    )
+    (property "Footprint" "" (at 121.6152 144.78 0)
+      (effects (font (size 1.27 1.27)) hide)
+    )
+    (property "Datasheet" "~" (at 120.65 140.97 0)
+      (effects (font (size 1.27 1.27)) hide)
+    )
+    (pin "1")
+    (pin "2")
+    (instances
+      (project "pcbV4"
+        (path "/499be7d4-fba5-4711-ae03-4b2682fa02d7"
+          (reference "C28") (unit 1)
+        )
+      )

Commit message: Update pcbV4 KiCad design
Parts:
- removed BB1: Conn_01x01_Pin, Connector_Wire:SolderWirePad_1x01_SMD_5x10mm, symbol Connector:Conn_01x01_Pin
- removed C27: 100nF, symbol Device:C
- removed R5: 200k, Resistor_SMD:R_0402_1005Metric, symbol Device:R
- removed U7: W25Q256JVFIQT, easyeda2kicad:SOIC-16_L10.3-W7.5-P1.27-LS10.3-BL, symbol battery:W25Q256JVFIQT
- added BT1: MY-2032-12, easyeda2kicad:BAT-SMD_MY-2032-12, symbol battery:MY-2032-12
- added C29: 22uF, symbol Device:C
- added C30: 100nF, symbol Device:C
- added JP1: SolderJumper_2_Open, symbol Jumper:SolderJumper_2_Open
- added Q2: AO3401A, easyeda2kicad:SOT-23_L2.9-W1.3-P1.90-LS2.4-BR, symbol battery:AO3401A
- added Q3, Q4: MMBT3904-TP, easyeda2kicad:SOT-23-3_L2.9-W1.3-P1.90-LS2.4-BR, symbol battery:MMBT3904-TP
- added R15, R16: 100k, symbol Device:R
- added R17: 660k, symbol Device:R
- added SW1: KMR221GLFS, easyeda2kicad:KEY-SMD_KMR2XXGXXX, symbol battery:KMR221GLFS
- added U9: W25Q256JVEIQTR, easyeda2kicad:WSON-8_L8.0-W6.10-P1.27-BL-EP, symbol battery:W25Q256JVEIQTR
- J3: value GND -> NRESET
Connections:
- net GND: now also BT1.2, C29.2, C30.2, Q3.2 (E), Q4.2 (E), U9.4 (GND), U9.9 (EP); no longer J3.1 (Pin_1)
- net MISO: now also U9.2 (DO(IO1))
- net MOSI: now also U9.5 (DI(IO0))
- net NRESET: now also J3.1 (Pin_1)
- net SCLK: now also U9.6 (CLK)
- net VDD: now also C30.1, JP1.2 (B), Q2.2 (S), R16.1, U9.3 (WP#(IO2)), U9.7 (HOLD#orRESET#(IO3)), U9.8 (VCC); no longer C21.1, L1.1, U4.1 (VOUTB)
- net W25_CS: now also U9.1 (~{CS})
- net bat+: now also BT1.1
- new net: C29.1, Q4.3 (C), R17.2, SW1.3
- new net: Q3.1 (B), Q4.1 (B), R16.2, SW1.1
- new net: Q2.1 (G), Q3.3 (C), R15.2
- new net npm_out: C21.1, JP1.1 (A), L1.1, Q2.3 (D), R15.1, R17.1, U4.1 (VOUTB)
- no-connect marks 23 -> 19
Other:
- note added: "PWR switch"

Commit message: Update pcbV4 KiCad design
Parts:
- removed R7, R8: 5k1, Resistor_SMD:R_0402_1005Metric, symbol Device:R
- removed USBC1: TYPE-C-31-M-12, easyeda2kicad:USB-C_SMD-TYPE-C-31-M-12_1, symbol npm:TYPE-C-31-M-12
- added R18, R5: 5k1, Resistor_SMD:R_0402_1005Metric, symbol Device:R
- added USB1: TYPE-C 16PFS 2JCB1.6-H6.5 IPX8, easyeda2kicad:USB-C-SMD_SHOUHAN_TYPE-C-16PFS-2JCB1.2-H6.5, symbol battery:TYPE-C16PFS2JCB1.6-H6.5IPX8
Connections:
- net GND: now also R18.2, R5.2, USB1.13 (EH), USB1.B12A1 (GND), USB1.B1A12 (GND)
- net VBUS: now also USB1.A4B9 (VBUS), USB1.A9B4 (VBUS)
- new net: R18.1, USB1.A5 (CC1)
- new net: R5.1, USB1.B5 (CC2)

Commit message: Update pcbV4 KiCad design
Parts:
- removed C28: 0.01uF, symbol Device:C
- removed C29: 22uF, symbol Device:C
- removed JP1: SolderJumper_2_Open, symbol Jumper:SolderJumper_2_Open
- removed OSC1: SX2M32.768KM20F30TNN, easyeda2kicad:OSC-SMD_4P-L2.5-W2.0-BL, symbol battery:SX2M32.768KM20F30TNN
- removed Q2: AO3401A, easyeda2kicad:SOT-23_L2.9-W1.3-P1.90-LS2.4-BR, symbol battery:AO3401A
- removed Q3, Q4: MMBT3904-TP, easyeda2kicad:SOT-23-3_L2.9-W1.3-P1.90-LS2.4-BR, symbol battery:MMBT3904-TP
- removed R15, R16: 100k, symbol Device:R
- removed R17: 660k, symbol Device:R
- removed U5: BS-08-B2AA020-R, easyeda2kicad:BAT-SMD_BS-08-B2AA016, symbol easyeda2kicad:BS-08-B2AA020-R
- removed USB1: TYPE-C 16PFS 2JCB1.6-H6.5 IPX8, easyeda2kicad:USB-C-SMD_SHOUHAN_TYPE-C-16PFS-2JCB1.2-H6.5, symbol battery:TYPE-C16PFS2JCB1.6-H6.5IPX8
- added H1, H2: MountingHole, MountingHole:MountingHole_2.2mm_M2, symbol Mechanical:MountingHole
- added LED1: 19-237/R6GHBHC-A07/2T, easyeda2kicad:LED-ARRAY-SMD_4P-L1.6-W1.6-BL-CW, symbol battery:19-237_R6GHBHC-A07_2T
- added R19: 1k, Resistor_SMD:R_0402_1005Metric, symbol Device:R
- added R7, R8: 5k1, Resistor_SMD:R_0402_1005Metric, symbol Device:R
- added TP3, TP4: TestPoint, TestPoint:TestPoint_Pad_D1.5mm, symbol Connector:TestPoint
- added USB2: USBC-0032IPX8-00, easyeda2kicad:TYPE-C-USB-SMD_USBC-0032IPX8-00, symbol battery:USBC-0032IPX8-00
- C30: footprint (none) -> Capacitor_SMD:C_0402_1005Metric
- R11, R12, R13, R14: footprint (none) -> Resistor_SMD:R_0402_1005Metric
- R18, R5: value 5k1 -> 1k
- TP1, TP2: footprint (none) -> TestPoint:TestPoint_Pad_D1.5mm
Connections:
- net npm_out is gone; now on net VDD: C21.1, L1.1, U4.1 (VOUTB)
- net BAT_MON: now also U3.15 (P1.07)
- net BAT_MON_EN: now also U3.25 (P2.08)
- net CHG: now also U3.27 (P2.10)
- net FCLK: now also U3.34 (P0.04)
- net GND: now also SW1.3, R7.1, R8.2, USB2.7 (EH), USB2.A12 (GND), USB2.B12 (GND); no longer R18.2, R5.2
- net MISO: now also TP3.1
- net MOSI: now also TP4.1
- net VBUS: now also USB2.B9 (VBUS)
- net VDD: now also LED1.4 (+)
- net W25_CS: now also U3.22 (P2.05)
- net NRF_BUTTON: now reaches SW1.1
- net NRF_BUTTON: now also U3.16 (P1.08)
- net at R18.1: now also LED1.2 (G-)
- net at R5.1: now also LED1.3 (B-)
- net LED_RED_DRAIN: now reaches U3.28 (P0.00)
- net LED_RED_DRAIN: now also R19.2
- net LED_GREEN_DRAIN: now reaches U3.29 (P0.01)
- net LED_GREEN_DRAIN: now also R18.2
- net LED_BLUE_DRAIN: now reaches U3.32 (P0.02)
- net LED_BLUE_DRAIN: now also R5.2
- net SCL: no longer names the net of U3.11 (P1.03)
- net SDA: no longer names the net of U3.10 (P1.02)
- new net: R7.2, USB2.A5 (CC1)
- new net: R8.1, USB2.B5 (CC2)
- new net: LED1.1 (R-), R19.1
- no-connect marks 19 -> 12
Other:
- note removed: "Crystal Oscillator 32.668KHz"
- note removed: "PWR switch"
- moved on the sheet: SW1, TP2, U3

Commit message: Update PCB design
Parts:
- added U5: ~, aer:ECG connectors, symbol RF_Module:ECG_Connector
Connections:
- net ECGN: now also U5. (ECG-)
- net ECGP: now also U5. (ECG-)
- net VBUS: now also USB2.A9 (VBUS)
- net VDD: now also LED1.2 (G-); no longer LED1.4 (+)
- net at R18.1: now also LED1.4 (+); no longer LED1.2 (G-)
Other:
- moved on the sheet: R18
Changed lines of the file:
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@@
     (stroke (width 0) (type default))
   )
+  (wire (pts (xy 384.81 106.68) (xy 386.08 106.68))
+    (stroke (width 0) (type default))
+  )
   (wire (pts (xy 370.84 212.725) (xy 373.38 212.725))
     (stroke (width 0) (type default))
@@
     (stroke (width 0) (type default))
   )
+  (wire (pts (xy 27.94 238.125) (xy 29.845 240.03))
+    (stroke (width 0) (type default))
+  )
   (wire (pts (xy 185.42 46.99) (xy 190.5 46.99))
     (stroke (width 0) (type default))
@@
     (stroke (width 0) (type default))
   )
+  (wire (pts (xy 27.94 219.075) (xy 27.94 238.125))
+    (stroke (width 0) (type default))
+  )
   (wire (pts (xy 33.02 223.52) (xy 36.195 223.52))
     (stroke (width 0) (type default))
@@
     (stroke (width 0) (type default))
   )
+  (wire (pts (xy 27.94 203.2) (xy 33.02 198.12))
+    (stroke (width 0) (type default))
+  )
   (wire (pts (xy 33.655 240.03) (xy 36.195 240.03))
     (stroke (width 0) (type default))
@@
     (stroke (width 0) (type default))
   )
+  (wire (pts (xy 251.46 97.155) (xy 255.27 97.155))
+    (stroke (width 0) (type default))
+  )
   (wire (pts (xy 388.62 167.64) (xy 388.62 171.45))
     (stroke (width 0) (type default))
@@
     (stroke (width 0) (type default))
   )
+  (wire (pts (xy 27.94 213.995) (xy 27.94 203.2))
+    (stroke (width 0) (type default))
+  )
   (wire (pts (xy 261.62 235.585) (xy 267.97 235.585))
     (stroke (width 0) (type default))
@@
     )
   )
-  (global_label "LED_GREEN_DRAIN" (shape input) (at 259.08 97.155 0) (fields_autoplaced)
-    (effects (font (size 1.27 1.27)) (justify left))
-    (property "Intersheetrefs" "${INTERSHEET_REFS}" (at 279.7419 97.155 0)
-      (effects (font (size 1.27 1.27)) (justify left) hide)
+  (global_label "LED_GREEN_DRAIN" (shape input) (at 228.6 97.155 180) (fields_autoplaced)
+    (effects (font (size 1.27 1.27)) (justify right))
+    (property "Intersheetrefs" "${INTERSHEET_REFS}" (at 207.9381 97.155 0)
+      (effects (font (size 1.27 1.27)) (justify right) hide)
     )
   )
@@
     )
   )
-  (symbol (lib_id "Device:R") (at 255.27 97.155 90) (unit 1)
+  (symbol (lib_id "Device:R") (at 232.41 97.155 270) (unit 1)
     (in_bom yes) (on_board yes) (dnp no) (fields_autoplaced)
-    (property "Reference" "R18" (at 255.27 91.44 90)
+    (property "Reference" "R18" (at 232.41 102.87 90)
       (effects (font (size 1.27 1.27)))
     )
-    (property "Value" "1k" (at 255.27 93.98 90)
+    (property "Value" "1k" (at 232.41 100.33 90)
       (effects (font (size 1.27 1.27)))
     )
-    (property "Footprint" "Resistor_SMD:R_0402_1005Metric" (at 255.27 98.933 90)
+    (property "Footprint" "Resistor_SMD:R_0402_1005Metric" (at 232.41 95.377 90)
       (effects (font (size 1.27 1.27)) hide)
     )
-    (property "Datasheet" "~" (at 255.27 97.155 0)
+    (property "Datasheet" "~" (at 232.41 97.155 0)
       (effects (font (size 1.27 1.27)) hide)
     )
@@
     )
   )
+  (symbol (lib_id "RF_Module:ECG_Connector") (at 22.86 216.535 90) (mirror x) (unit 1)
+    (in_bom yes) (on_board yes) (dnp no)
+    (property "Reference" "U5" (at 22.86 222.25 90)
+      (effects (font (size 1.27 1.27)))
+    )
+    (property "Value" "~" (at 22.86 216.535 0)
+      (effects (font (size 1.27 1.27)))
+    )
+    (property "Footprint" "aer:ECG connectors" (at 22.86 216.535 0)
+      (effects (font (size 1.27 1.27)) hide)
+    )
+    (property "Datasheet" "" (at 22.86 216.535 0)
+      (effects (font (size 1.27 1.27)) hide)
+    )
+    (pin "")
+    (pin "")
+    (instances
+      (project "pcbV4"
+        (path "/499be7d4-fba5-4711-ae03-4b2682fa02d7"
+          (reference "U5") (unit 1)
+        )
+      )
+    )
+  )
   (symbol (lib_id "power:GND") (at 359.41 116.84 0) (unit 1)
     (in_bom yes) (on_board yes) (dnp no) (fields_autoplaced)
@@
     )
   )
-  (symbol (lib_id "power:VDD") (at 236.22 97.155 0) (unit 1)
+  (symbol (lib_id "power:VDD") (at 255.27 97.155 0) (unit 1)
     (in_bom yes) (on_board yes) (dnp no) (fields_autoplaced)
-    (property "Reference" "#PWR032" (at 236.22 100.965 0)
+    (property "Reference" "#PWR032" (at 255.27 100.965 0)
       (effects (font (size 1.27 1.27)) hide)
     )
-    (property "Value" "VDD" (at 236.22 92.71 0)
+    (property "Value" "VDD" (at 255.27 92.71 0)
       (effects (font (size 1.27 1.27)))
     )
-    (property "Footprint" "" (at 236.22 97.155 0)
+    (property "Footprint" "" (at 255.27 97.155 0)
       (effects (font (size 1.27 1.27)) hide)
     )
-    (property "Datasheet" "" (at 236.22 97.155 0)
+    (property "Datasheet" "" (at 255.27 97.155 0)
       (effects (font (size 1.27 1.27)) hide)
     )
